Commit message: change the package name and input physics data estimated

File: elite_robot_description/urdf/cs66_macro.urdf.xacro (robot description, xacro)
@@ -1,10 +1,10 @@
 <?xml version="1.0"?>
 <robot xmlns:xacro="http://www.ros.org/wiki/xacro">
-    <xacro:macro name="insert_robot" params="prefix parent *origin">
+    <xacro:macro name="insert_robot" params="prefix model parent *origin">
         <link name="${prefix}base_link">
             <visual>
                 <origin xyz="0 0 0" rpy="0 0 0"/>
                 <geometry>
-                    <mesh filename="package://cs66_description/meshes/visual/base.dae" scale="1 1 1"/>
+                    <mesh filename="package://elite_robot_description/meshes/${model}/visual/base.dae" scale="1 1 1"/>
                 </geometry>
             </visual>
@@ -12,11 +12,11 @@
                 <origin xyz="0 0 0" rpy="0 0 0"/>
                 <geometry>
-                    <mesh filename="package://cs66_description/meshes/visual/base.dae" scale="1 1 1"/>
+                    <mesh filename="package://elite_robot_description/meshes/${model}/collison/base.stl" scale="1 1 1"/>
                 </geometry>
             </collision>
             <inertial>
-                <origin xyz="0 0 0" rpy="0 0 0"/>
-                <mass value="1.0"/>
-                <inertia ixx="1.0" ixy="0" ixz="0" iyy="1.0" iyz="0" izz="1.0"/>
+                <origin xyz="0 0 0" rpy="0 0 0.042"/>
+                <mass value="1.753476"/>
+                <inertia ixx="0.003313" ixy="0" ixz="0" iyy="0.003312" iyz="0" izz="0.004254"/>
             </inertial>
         </link>
@@ -30,5 +30,5 @@
                 <origin xyz="0 0 0" rpy="0 0 0"/>
                 <geometry>
-                    <mesh filename="package://cs66_description/meshes/visual/link1.dae" scale="1 1 1"/>
+                    <mesh filename="package://elite_robot_description/meshes/${model}/visual/link1.dae" scale="1 1 1"/>
                 </geometry>
             </visual>
@@ -36,11 +36,11 @@
                 <origin xyz="0 0 0" rpy="0 0 0"/>
                 <geometry>
-                    <mesh filename="package://cs66_description/meshes/visual/link1.dae" scale="1 1 1"/>
+                    <mesh filename="package://elite_robot_description/meshes/${model}/collison/link1.stl" scale="1 1 1"/>
                 </geometry>
             </collision>
             <inertial>
-                <origin xyz="0 0 0" rpy="0 0 0"/>
-                <mass value="1.0"/>
-                <inertia ixx="1.0" ixy="0" ixz="0" iyy="1.0" iyz="0" izz="1.0"/>
+                <origin xyz="0 -0.009 0.072" rpy="0 0 0"/>
+                <mass value="2.431303"/>
+                <inertia ixx="0.006723" ixy="0" ixz="0.000001" iyy="0.006327" iyz="0.000046" izz="0.005198"/>
             </inertial>
         </link>
@@ -56,5 +56,5 @@
                 <origin xyz="0 0 0" rpy="0 0 0"/>
                 <geometry>
-                    <mesh filename="package://cs66_description/meshes/visual/link2.dae" scale="1 1 1"/>
+                    <mesh filename="package://elite_robot_description/meshes/${model}/visual/link2.dae" scale="1 1 1"/>
                 </geometry>
             </visual>
@@ -62,11 +62,11 @@
                 <origin xyz="0 0 0" rpy="0 0 0"/>
                 <geometry>
-                    <mesh filename="package://cs66_description/meshes/visual/link2.dae" scale="1 1 1"/>
+                    <mesh filename="package://elite_robot_description/meshes/${model}/collison/link2.stl" scale="1 1 1"/>
                 </geometry>
             </collision>
             <inertial>
-                <origin xyz="0 0 0" rpy="0 0 0"/>
-                <mass value="1.0"/>
-                <inertia ixx="1.0" ixy="0" ixz="0" iyy="1.0" iyz="0" izz="1.0"/>
+                <origin xyz="0.199 0.073 0.000" rpy="0 0 0"/>
+                <mass value="10.308232"/>
+                <inertia ixx="0.027417" ixy="-0.000970" ixz="0.000007" iyy="0.233058" iyz="0" izz="0.240741"/>
             </inertial>
         </link>
@@ -82,5 +82,5 @@
                 <origin xyz="0 0 0" rpy="0 0 0"/>
                 <geometry>
-                    <mesh filename="package://cs66_description/meshes/visual/link3.dae" scale="1 1 1"/>
+                    <mesh filename="package://elite_robot_description/meshes/${model}/visual/link3.dae" scale="1 1 1"/>
                 </geometry>
             </visual>
@@ -88,11 +88,11 @@
                 <origin xyz="0 0 0" rpy="0 0 0"/>
                 <geometry>
-                    <mesh filename="package://cs66_description/meshes/visual/link3.dae" scale="1 1 1"/>
+                    <mesh filename="package://elite_robot_description/meshes/${model}/collison/link3.stl" scale="1 1 1"/>
                 </geometry>
             </collision>
             <inertial>
-                <origin xyz="0 0 0" rpy="0 0 0"/>
-                <mass value="1.0"/>
-                <inertia ixx="1.0" ixy="0" ixz="0" iyy="1.0" iyz="0" izz="1.0"/>
+                <origin xyz="0.194 -0.058 0.000" rpy="0 0 0"/>
+                <mass value="5.342591"/>
+                <inertia ixx="0.008507" ixy="0.005298" ixz="0.000001" iyy="0.092157" iyz="0" izz="0.094359"/>
             </inertial>
         </link>
@@ -108,5 +108,5 @@
                 <origin xyz="0 0 0" rpy="0 0 0"/>
                 <geometry>
-                    <mesh filename="package://cs66_description/meshes/visual/link4.dae" scale="1 1 1"/>
+                    <mesh filename="package://elite_robot_description/meshes/${model}/visual/link4.dae" scale="1 1 1"/>
                 </geometry>
             </visual>
@@ -114,11 +114,11 @@
                 <origin xyz="0 0 0" rpy="0 0 0"/>
                 <geometry>
-                    <mesh filename="package://cs66_description/meshes/visual/link4.dae" scale="1 1 1"/>
+                    <mesh filename="package://elite_robot_description/meshes/${model}/collison/link4.stl" scale="1 1 1"/>
                 </geometry>
             </collision>
             <inertial>
-                <origin xyz="0 0 0" rpy="0 0 0"/>
-                <mass value="1.0"/>
-                <inertia ixx="1.0" ixy="0" ixz="0" iyy="1.0" iyz="0" izz="1.0"/>
+                <origin xyz="0 0.064 0.006" rpy="0 0 0"/>
+                <mass value="1.119554"/>
+                <inertia ixx="0.002172" ixy="0" ixz="0" iyy="0.001469" iyz="-0.000062" izz="0.001640"/>
             </inertial>
         </link>
@@ -134,5 +134,5 @@
                 <origin xyz="0 0 0" rpy="0 0 0"/>
                 <geometry>
-                    <mesh filename="package://cs66_description/meshes/visual/link5.dae" scale="1 1 1"/>
+                    <mesh filename="package://elite_robot_description/meshes/${model}/visual/link5.dae" scale="1 1 1"/>
                 </geometry>
             </visual>
@@ -140,11 +140,11 @@
                 <origin xyz="0 0 0" rpy="0 0 0"/>
                 <geometry>
-                    <mesh filename="package://cs66_description/meshes/visual/link5.dae" scale="1 1 1"/>
+                    <mesh filename="package://elite_robot_description/meshes/${model}/collison/link5.stl" scale="1 1 1"/>
                 </geometry>
             </collision>
             <inertial>
-                <origin xyz="0 0 0" rpy="0 0 0"/>
-                <mass value="1.0"/>
-                <inertia ixx="1.0" ixy="0" ixz="0" iyy="1.0" iyz="0" izz="1.0"/>
+                <origin xyz="0 -0.006 0.042" rpy="0 0 0"/>
+                <mass value="0.801370"/>
+                <inertia ixx="0.001175" ixy="0" ixz="0" iyy="0.000723" iyz="0.000009" izz="0.001108"/>
             </inertial>
         </link>
@@ -160,5 +160,5 @@
                 <origin xyz="0 0 0" rpy="0 0 0"/>
                 <geometry>
-                    <mesh filename="package://cs66_description/meshes/visual/link6.dae" scale="1 1 1"/>
+                    <mesh filename="package://elite_robot_description/meshes/${model}/visual/link6.dae" scale="1 1 1"/>
                 </geometry>
             </visual>
@@ -166,11 +166,11 @@
                 <origin xyz="0 0 0" rpy="0 0 0"/>
                 <geometry>
-                    <mesh filename="package://cs66_description/meshes/visual/link6.dae" scale="1 1 1"/>
+                    <mesh filename="package://elite_robot_description/meshes/${model}/collison/link6.stl" scale="1 1 1"/>
                 </geometry>
             </collision>
             <inertial>
-                <origin xyz="0 0 0" rpy="0 0 0"/>
-                <mass value="1.0"/>
-                <inertia ixx="1.0" ixy="0" ixz="0" iyy="1.0" iyz="0" izz="1.0"/>
+                <origin xyz="0 0.021 0.001" rpy="0 0 0"/>
+                <mass value="0.243472"/>
+                <inertia ixx="0.000124" ixy="0" ixz="0" iyy="0.000173" iyz="0" izz="0.000119"/>
             </inertial>
         </link>

Commit message: Add package elite_robot_hardware_interface

File: elite_robot_description/urdf/cs66_macro.urdf.xacro (robot description, xacro)
@@ -1,5 +1,5 @@
 <?xml version="1.0"?>
 <robot xmlns:xacro="http://www.ros.org/wiki/xacro">
-    <xacro:macro name="insert_robot" params="prefix model parent *origin">
+    <xacro:macro name="insert_robot" params="prefix model parent *origin robot_ip dashboard_port controller_port rtsi_port">
         <link name="${prefix}base_link">
             <visual>
@@ -194,4 +194,11 @@
             <origin xyz="0 0.043 0" rpy="${-pi/2} 0 0"/>
         </joint>
+        <xacro:insert_ros2_control
+            prefix="${prefix}"
+            robot_ip="${robot_ip}"
+            dashboard_port="${dashboard_port}"
+            controller_port="${controller_port}"
+            rtsi_port="${rtsi_port}"
+        />
     </xacro:macro>
 </robot>

File: elite_robot_description/urdf/robot.urdf.xacro (robot description, xacro)
@@ -4,6 +4,19 @@
     <xacro:include filename="$(find elite_robot_description)/urdf/$(arg robot_model)_macro.urdf.xacro"/>
     <xacro:include filename="$(find elite_robot_description)/urdf/$(arg robot_model)_gazebo.urdf.xacro"/>
+    <xacro:include filename="$(find elite_robot_description)/urdf/$(arg robot_model)_ros2_control.urdf.xacro"/>
     <link name="world" />
-    <xacro:insert_robot prefix="" model="cs66" parent="world">
+    <xacro:arg name="robot_ip" default="127.0.0.1"/>
+    <xacro:arg name="dashboard_port" default="29999"/>
+    <xacro:arg name="controller_port" default="30001"/>
+    <xacro:arg name="rtsi_port" default="30004"/>
+    <xacro:insert_robot
+        prefix=""
+        model="cs66"
+        parent="world"
+        robot_ip="$(arg robot_ip)"
+        dashboard_port="$(arg dashboard_port)"
+        controller_port="$(arg controller_port)"
+        rtsi_port="$(arg rtsi_port)"
+    >
         <origin xyz="0 0 0" rpy="0 0 0"/>
     </xacro:insert_robot>
